File: AVR_ISP_USB_TQFP.kicad_pcb (KiCad board)
At the start: 2 copper layers, 47 x 20 mm, 22 parts, among them CON1 USB-MICRO-B, IC1 ATMEGA8-AI, P1 CONN_02X05, P2 CONN_01X01, P3 CONN_01X01, X1 CRYSTAL

Commit message: final
Parts:
- added P4: CONN_01X01, Connect:1pin, F.Cu at (143.0, 103.5)
- added P5: CONN_01X01, Connect:1pin, F.Cu at (143.0, 88.5)
- added R6: 1k, Resistors_SMD:R_0603_HandSoldering, F.Cu at (142.6, 91.8)
- added R7: 1k, Resistors_SMD:R_0603_HandSoldering, F.Cu at (137.4, 104.1)
- D3, D4: value ZENER -> 3.6V
- X1: value CRYSTAL -> 12MHz
- moved D1 1.52 mm to (145.5, 88.6), turned to 90 degrees
- moved D2 1.42 mm to (145.4, 103.4), turned to 90 degrees
- moved P3 0.50 mm to (109.5, 103.5)
Connections:
- D1 pad 1: VCC -> Net-(D1-Pad1)
- D2 pad 1: VCC -> Net-(D2-Pad1)
Routing:
- net Net-(D2-Pad1): track 0.00 -> 8.74 mm
- net Net-(D1-Pad1): track 0.00 -> 4.65 mm
- net Net-(D1-Pad2): track 8.28 -> 12.5 mm
- net Net-(IC1-Pad14): track 34.7 -> 32.3 mm
- net VCC: track 120.4 -> 118.2 mm
- net Net-(D2-Pad2): track 25.8 -> 24.2 mm
- net Net-(IC1-Pad25): track 31.0 -> 31.8 mm
- net Net-(IC1-Pad15): track 23.1 -> 23.7 mm
Other:
- board text added: "ExploreEmbedded.com"
- board text added: "USBasp"

Commit message: final_v1
Routing:
- net Net-(IC1-Pad29): track 29.6 -> 53.5 mm
- net GND: track 110.6 -> 113.6 mm
- net Net-(IC1-Pad25): track 31.8 -> 34.0 mm
- net Net-(IC1-Pad14): track 32.3 -> 33.8 mm
