File: _autosave-AVR_ISP_USB_TQFP.kicad_pcb (KiCad board)
At the start: 2 copper layers, 47 x 20 mm, 26 parts, among them CON1 USB-MICRO-B, IC1 ATMEGA8-AI, P1 CONN_02X05, P2 CONN_01X01, P3 CONN_01X01, P4 CONN_01X01, P5 CONN_01X01, X1 12MHz

Commit message: Final Gerber
Final gerber data generated
Other:
- board text added: "Explore USBasp"
- board text removed: "USBasp"
